File: KiCad/final/attiny13ir.kicad_pcb (KiCad board)
At the start: 2 copper layers, 20.8 x 29.3 mm, 9 parts, among them J1 Notch, J2 EXP2, J3 PIN29, U1 ATtiny13A-SU

Commit message: minor fixes
Parts:
- moved C1 11.2 mm to (105.4, 98.0), turned to 180 degrees
- moved J2 10.5 mm to (106.4, 100.8), turned to 90 degrees
Routing:
- net GND: track 84.9 -> 7.45 mm
- net +5V: track 30.6 -> 27.2 mm
