File: KiCad/testing/attiny13ir.sch (KiCad schematic (older format))
At the start: 12 parts, among them J1 Notch, J2 EXP2, J3 PIN29, J4 ICSP, SW1 Test switch, U1 ATtiny13A-SU

Commit message: minor fixes
Parts:
- R2: value 10k -> 1k
Changed lines of the file:
@@
 P 2700 3300
 F 0 "R2" H 2770 3346 50  0000 L CNN
-F 1 "10k" H 2770 3255 50  0000 L CNN
+F 1 "1k" H 2770 3255 50  0000 L CNN
 F 2 "Resistor_SMD:R_0805_2012Metric_Pad1.15x1.40mm_HandSolder" V 2630 3300 50  0001 C CNN
 F 3 "~" H 2700 3300 50  0001 C CNN
